File: bento-board-2/SUB-00156 REV00 20260424/Addressable RGB LED.kicad_sch (KiCad schematic)
At the start: 9 parts, among them U3 ${ALTIUM_VALUE}

Commit message: Add Bento Board 2 REV00 KiCad source files
Parts:
- C12, C6, C7, R22: FOOTPRINT 0603 (1608 Metric) -> (none)
- D5: FOOTPRINT 3228 -> (none)
- R7: FOOTPRINT R0603 -> (none)
- TP11, TP13: footprint Library:TP-SM-39MILC -> (none)
- U3: FOOTPRINT SOT23-5 -> (none)
