File: bento-board-2/SUB-00156 REV00 20260424/Buzzer.kicad_sch (KiCad schematic)
At the start: 6 parts, among them Q1 ${ALTIUM_VALUE}

Commit message: Add Bento Board 2 REV00 KiCad source files
Parts:
- LS1: FOOTPRINT PKLCS_472X472 -> (none)
- Q1: FOOTPRINT SOT23 -> (none)
- R39, R40, R408: FOOTPRINT 0603 (1608 Metric) -> (none)
- TP401: footprint Library:TP-SM-39MILC -> (none)
