File: bento-board-2/SUB-00156 REV00 20260424/ESP32-C3 RFSoC.kicad_sch (KiCad schematic)
At the start: 22 parts, among them J3 ${ALTIUM_VALUE}, SW2 ${ALTIUM_VALUE}, U5 ${ALTIUM_VALUE}

Commit message: Add Bento Board 2 REV00 KiCad source files
Parts:
- C8, C9, R10, R11, R12, R2, R24, R26, R27, R28, R29, R8, R9: FOOTPRINT 0603 (1608 Metric) -> (none)
- D2: FOOTPRINT 0603 -> (none)
- ESP32-RST, ESP32_3.3V, ESP32_RX, ESP32_TX, ESP_GND: footprint Library:TP-SM-39MILC -> (none)
- J3: FOOTPRINT TC2050-IDC -> (none)
- SW2: FOOTPRINT PTS810 -> (none)
Other:
- note added: "The J3 (TC2050-IDC) interface definition"
- note added: "is not the SWD standard connection method."
