File: bento-board-2/SUB-00156 REV00 20260424/Mechanical.kicad_sch (KiCad schematic)
At the start: 16 parts

Commit message: Add Bento Board 2 REV00 KiCad source files
Parts:
- BoardIDlabel1: footprint Library:Laebl_12_8mm -> (none)
- PCB1: footprint PCB Part Number -> (none)
- PLTTestedlabel1: footprint Library:Laebl_24_12mm -> (none)
- TP10, TP21, TP33, TP44: footprint Library:TP-SM-39MILC -> (none)
