File: bento-board-2/SUB-00156 REV00 20260424/Power.kicad_sch (KiCad schematic)
At the start: 21 parts, among them U6 ${ALTIUM_VALUE}

Commit message: Add Bento Board 2 REV00 KiCad source files
Parts:
- C901: FOOTPRINT C1210 -> (none)
- C902, FB901, R901, R903, R904, R905, R906, R907, R908, R909, R910, R911, R912, R932: FOOTPRINT 0603 (1608 Metric) -> (none)
- D901: FOOTPRINT SMA -> (none)
- D902: FOOTPRINT 0603 -> (none)
- S1: footprint Library:JS202011JAQN -> (none)
- TP901, TP902: footprint Library:TP-SM-39MILC -> (none)
- U6: FOOTPRINT TO-263 (DDPAK-3) -> (none)
