File: bento-board-2/SUB-00156 REV00 20260424/Qwiic.kicad_sch (KiCad schematic)
At the start: 10 parts, among them J4 ${ALTIUM_VALUE}, J5 ${ALTIUM_VALUE}

Commit message: Add Bento Board 2 REV00 KiCad source files
Parts:
- C10, C11, R13, R14, R15, R16: FOOTPRINT 0603 (1608 Metric) -> (none)
- I2C_SCL, I2C_SDA: footprint Library:TP-SM-39MILC -> (none)
- J4, J5: footprint Library:16766 -> (none)
