File: bento-board-2/SUB-00156 REV00 20260424/Relay.kicad_sch (KiCad schematic)
At the start: 9 parts, among them K1 ${ALTIUM_VALUE}, U4 ${ALTIUM_VALUE}

Commit message: Add Bento Board 2 REV00 KiCad source files
Parts:
- K1: FOOTPRINT 1462042-8 -> (none)
- R20: FOOTPRINT 0603 (1608 Metric) -> (none)
- TP101, TP102, TP103, TP201, TP202, TP203: footprint Library:TP-SM-39MILC -> (none)
- U4: FOOTPRINT 20-SOIC (0.295", 7.50mm Width) -> (none)
