File: bento-board-2/SUB-00156 REV00 20260424/Sensor.kicad_sch (KiCad schematic)
At the start: 2 parts, among them U30 ${ALTIUM_VALUE}

Commit message: Add Bento Board 2 REV00 KiCad source files
Parts:
- R21: FOOTPRINT 0603 (1608 Metric) -> (none)
- U30: FOOTPRINT 8-LGA (2.5x2.5) -> (none)
