File: bento-board-2/SUB-00156 REV00 20260424/Type-C.kicad_sch (KiCad schematic)
At the start: 16 parts, among them J51 ${ALTIUM_VALUE}

Commit message: Add Bento Board 2 REV00 KiCad source files
Parts:
- C51, R52: FOOTPRINT 1206 (3216 Metric) -> (none)
- C52, C53, FB1, R51, R53: FOOTPRINT 0603 (1608 Metric) -> (none)
- D51: FOOTPRINT 2-XDFN -> (none)
- GND, RP_USB_N, RP_USB_P, TP53, TP54, TP55: footprint Library:TP-SM-39MILC -> (none)
- J51: FOOTPRINT 10159872-00011LF -> (none)
