File: bento-board-2/SUB-00156 REV00 20260424/mikroBUS.kicad_sch (KiCad schematic)
At the start: 8 parts, among them J2 ${ALTIUM_VALUE}

Commit message: Add Bento Board 2 REV00 KiCad source files
Parts:
- J2: FOOTPRINT MIKROE-4319 -> (none)
- R17, R18, R19: FOOTPRINT 0603 (1608 Metric) -> (none)
- SCI1_RXD, SCI1_TXD, TP2, TP3: footprint Library:TP-SM-39MILC -> (none)
